Commit message: x02a全身sim2real测试ok

File: legged_lab/assets/droid/x02a/x02a.urdf (robot description, URDF)
Before this commit: robot x02a, 47 links, 46 joints
Links:
- link L_elbow_link: geometry collision cylinder length=0.35 radius=0.03; visual mesh filename=meshes/L_elbow_link.STL
- link L_shoulder_roll_link: geometry collision cylinder length=0.08 radius=0.04; visual mesh filename=meshes/L_shoulder_roll_link.STL
- link L_shoulder_yaw_link: geometry collision cylinder length=0.1 radius=0.04; visual mesh filename=meshes/L_shoulder_yaw_link.STL
- link R_elbow_link: geometry collision cylinder length=0.35 radius=0.03; visual mesh filename=meshes/R_elbow_link.STL
- link R_shoulder_roll_link: geometry collision cylinder length=0.08 radius=0.04; visual mesh filename=meshes/R_shoulder_roll_link.STL
- link R_shoulder_yaw_link: geometry collision cylinder length=0.1 radius=0.04; visual mesh filename=meshes/R_shoulder_yaw_link.STL
Joints:
- joint L_elbow: origin xyz=0 -0.01 0.148 rpy=1.5708 -3.1415 1.5708 -> xyz=0 -0.01 0.148 rpy=1.5708 -1.5708 1.5708; type fixed -> revolute
- joint L_shoulder_pitch: origin xyz=0 0.14043 0.29123 rpy=1.0 1.0 2.6 -> xyz=0 0.14043 0.29123 rpy=0 1.309 1.5708; type fixed -> revolute
- joint L_shoulder_roll: type fixed -> revolute
- joint L_shoulder_yaw: type fixed -> revolute
- joint R_elbow: origin xyz=0 0.01 0.148 rpy=1.5708 0 1.5708 -> xyz=0 0.01 0.148 rpy=1.5708 -1.5708 1.5708; type fixed -> revolute
- joint R_shoulder_pitch: origin xyz=0 -0.14043 0.29123 rpy=-1.0 1.0 -2.6 -> xyz=0 -0.14043 0.29123 rpy=0 1.309 -1.5708; type fixed -> revolute
- joint R_shoulder_roll: type fixed -> revolute
- joint R_shoulder_yaw: type fixed -> revolute
