Commit message: 简化x2r模型碰撞体

File: legged_lab/assets/droid/x2r10/x2r10.urdf (robot description, URDF)
Before this commit: robot x2r10, 23 links, 22 joints
Links:
- link L_ankle_pitch_link: geometry collision box size=0.29 0.09 0.025; visual mesh filename=meshes/L_ankle_pitch_link.STL
- link L_elbow_pitch_link: geometry collision sphere radius=0.038; visual mesh filename=meshes/L_elbow_pitch_link.STL
- link L_hip_pitch_link: geometry collision cylinder length=0.25 radius=0.07; visual mesh filename=meshes/L_hip_pitch_link.STL
- link L_knee_pitch_link: geometry collision cylinder length=0.2 radius=0.05; visual mesh filename=meshes/L_knee_pitch_link.STL
- link L_shoulder_pitch_link: geometry visual mesh filename=meshes/L_shoulder_pitch_link.STL
- link L_shoulder_roll_link: geometry collision cylinder length=0.08 radius=0.04; visual mesh filename=meshes/L_shoulder_roll_link.STL
- link L_shoulder_yaw_link: geometry collision cylinder length=0.08 radius=0.04; visual mesh filename=meshes/L_shoulder_yaw_link.STL
- link R_ankle_pitch_link: geometry collision box size=0.29 0.09 0.025; visual mesh filename=meshes/R_ankle_pitch_link.STL
- link R_elbow_pitch_link: geometry collision sphere radius=0.038; visual mesh filename=meshes/R_elbow_pitch_link.STL
- link R_hip_pitch_link: geometry collision cylinder length=0.25 radius=0.07; visual mesh filename=meshes/R_hip_pitch_link.STL
- link R_knee_pitch_link: geometry collision cylinder length=0.2 radius=0.05; visual mesh filename=meshes/R_knee_pitch_link.STL
- link R_shoulder_pitch_link: geometry visual mesh filename=meshes/R_shoulder_pitch_link.STL
- link R_shoulder_roll_link: geometry collision cylinder length=0.08 radius=0.04; visual mesh filename=meshes/R_shoulder_roll_link.STL
- link R_shoulder_yaw_link: geometry collision cylinder length=0.08 radius=0.04; visual mesh filename=meshes/R_shoulder_yaw_link.STL
- link head_link: geometry collision sphere radius=0.12; visual mesh filename=meshes/head_link.STL
- link logo_link: geometry visual mesh filename=meshes/logo_link.STL
- link pelvis_link: geometry collision box size=0.25 0.3 0.4; visual mesh filename=meshes/pelvis_link.STL
- link torso_link: geometry visual mesh filename=meshes/torso_link.STL
- link waist_yaw_link: geometry visual mesh filename=meshes/waist_yaw_link.STL

File: legged_lab/assets/droid/x2rw10/x2rw10.urdf (robot description, URDF)
Before this commit: robot x2rw10, 23 links, 22 joints
Links:
- link L_ankle_pitch_link: geometry collision box size=0.29 0.09 0.025; visual mesh filename=meshes/L_ankle_pitch_link.STL
- link L_elbow_pitch_link: geometry collision sphere radius=0.038; visual mesh filename=meshes/L_elbow_pitch_link.STL
- link L_hip_pitch_link: geometry collision cylinder length=0.25 radius=0.07; visual mesh filename=meshes/L_hip_pitch_link.STL
- link L_knee_pitch_link: geometry collision cylinder length=0.2 radius=0.05; visual mesh filename=meshes/L_knee_pitch_link.STL
- link L_shoulder_pitch_link: geometry visual mesh filename=meshes/L_shoulder_pitch_link.STL
- link L_shoulder_roll_link: geometry collision cylinder length=0.08 radius=0.04; visual mesh filename=meshes/L_shoulder_roll_link.STL
- link L_shoulder_yaw_link: geometry collision cylinder length=0.08 radius=0.04; visual mesh filename=meshes/L_shoulder_yaw_link.STL
- link R_ankle_pitch_link: geometry collision box size=0.29 0.09 0.025; visual mesh filename=meshes/R_ankle_pitch_link.STL
- link R_elbow_pitch_link: geometry collision sphere radius=0.038; visual mesh filename=meshes/R_elbow_pitch_link.STL
- link R_hip_pitch_link: geometry collision cylinder length=0.25 radius=0.07; visual mesh filename=meshes/R_hip_pitch_link.STL
- link R_knee_pitch_link: geometry collision cylinder length=0.2 radius=0.05; visual mesh filename=meshes/R_knee_pitch_link.STL
- link R_shoulder_pitch_link: geometry visual mesh filename=meshes/R_shoulder_pitch_link.STL
- link R_shoulder_roll_link: geometry collision cylinder length=0.08 radius=0.04; visual mesh filename=meshes/R_shoulder_roll_link.STL
- link R_shoulder_yaw_link: geometry collision cylinder length=0.08 radius=0.04; visual mesh filename=meshes/R_shoulder_yaw_link.STL
- link head_link: geometry collision sphere radius=0.12; visual mesh filename=meshes/head_link.STL
- link logo_link: geometry visual mesh filename=meshes/logo_link.STL
- link pelvis_link: geometry collision box size=0.25 0.3 0.4; visual mesh filename=meshes/pelvis_link.STL
- link torso_link: geometry visual mesh filename=meshes/torso_link.STL
- link waist_yaw_link: geometry visual mesh filename=meshes/waist_yaw_link.STL
