Commit message: 更新x2模型为10自由度，sim2real测试ok

File: legged_lab/assets/droid/x2/x2.urdf (robot description, URDF)
Before this commit: robot x2, 47 links, 46 joints
Links:
- link pelvis_link: mass 9.129 -> 0.129
Joints:
- joint L_ankle_pitch: limit lower=-1.2217 upper=1.2217 effort=30 velocity=10 -> lower=-0.6 upper=0.6 effort=30 velocity=10
- joint L_elbow_pitch: origin xyz=0 -0.01 0.148 rpy=1.5708 -1.5708 1.5708 -> xyz=0 -0.01 0.148 rpy=1.5708 -2.2 1.5708; type revolute -> fixed
- joint L_shoulder_pitch: type revolute -> fixed
- joint L_shoulder_roll: type revolute -> fixed
- joint L_shoulder_yaw: type revolute -> fixed
- joint R_ankle_pitch: limit lower=-1.2217 upper=1.2217 effort=30 velocity=10 -> lower=-0.6 upper=0.6 effort=30 velocity=10
- joint R_elbow_pitch: origin xyz=0 0.01 0.148 rpy=1.5708 -1.5708 1.5708 -> xyz=0 0.01 0.148 rpy=1.5708 -0.9416 1.5708; type revolute -> fixed
- joint R_shoulder_pitch: type revolute -> fixed
- joint R_shoulder_roll: type revolute -> fixed
- joint R_shoulder_yaw: type revolute -> fixed

Commit message: 区分x2不同构型的机器人模型

File: legged_lab/assets/droid/x2/x2.urdf (robot description, URDF)
Before this commit: robot x2, 47 links, 46 joints
Links:
- added link world
- link L_ankle_pitch_link: geometry collision mesh filename=meshes/L_ankle_pitch_link.STL; visual mesh filename=meshes/L_ankle_pitch_link.STL
- link R_ankle_pitch_link: geometry collision mesh filename=meshes/R_ankle_pitch_link.STL; visual mesh filename=meshes/R_ankle_pitch_link.STL
Joints:
- added joint pelvis_link: type floating, parent world, child pelvis_link
- joint L_elbow_pitch: origin xyz=0 -0.01 0.148 rpy=1.5708 -2.2 1.5708 -> xyz=0 -0.01 0.148 rpy=1.5708 -1.5708 1.5708; type fixed -> revolute
- joint L_forearm_yaw: type fixed -> revolute
- joint L_shoulder_pitch: origin xyz=0 0.14043 0.29123 rpy=0 1.309 1.5708 -> xyz=0 0.14043 0.29123 rpy=0 1.5708 1.5708; type fixed -> revolute
- joint L_shoulder_roll: origin xyz=0 0 0.0575 rpy=-1.5708 0.2618 0 -> xyz=0 0 0.0575 rpy=-1.5708 0 0; type fixed -> revolute
- joint L_shoulder_yaw: type fixed -> revolute
- joint R_elbow_pitch: origin xyz=0 0.01 0.148 rpy=1.5708 -0.9416 1.5708 -> xyz=0 0.01 0.148 rpy=1.5708 -1.5708 1.5708; type fixed -> revolute
- joint R_forearm_yaw: type fixed -> revolute
- joint R_shoulder_pitch: origin xyz=0 -0.14043 0.29123 rpy=0 1.309 -1.5708 -> xyz=0 -0.14043 0.29123 rpy=0 1.5708 -1.5708; type fixed -> revolute
- joint R_shoulder_roll: origin xyz=0 0 0.0575 rpy=-1.5708 0.2618 0 -> xyz=0 0 0.0575 rpy=-1.5708 0 0; type fixed -> revolute
- joint R_shoulder_yaw: type fixed -> revolute
