Commit message: 调整机器人模型文件目录组织结构

File: legged_lab/assets/droid/x2r/x2r10/x2r10.urdf (robot description, URDF)
Before this commit: robot x2r10, 23 links, 22 joints
Links:
- removed link head_link
- added link Head_yaw_link, mass 1.67; collision sphere radius=0.12; visual mesh filename=meshes/Head_yaw_link.STL
Joints:
- joint head: child head_link -> Head_yaw_link
