Commit message: E1 Sim2Real测试ok

File: legged_lab/assets/droid/E1-1/E1.urdf (robot description, URDF)
Before this commit: robot E1_1105, 31 links, 30 joints
Joints:
- joint waist_yaw_joint: type fixed -> revolute

File: legged_lab/assets/droid/E1/E1.urdf (robot description, URDF)
Before this commit: robot E1_1105, 26 links, 25 joints
Links:
- added link head_pitch_link, mass 0.4; collision box size=0.04 0.04 0.04; visual mesh filename=meshes/head_pitch_link.STL
- added link head_yaw_link, mass 1; collision box size=0.10 0.10 0.10; visual mesh filename=meshes/head_yaw_link.STL
- added link left_wrist_yaw_link, mass 0.2; collision sphere radius=0.03; visual mesh filename=meshes/left_wrist_yaw_link.STL
- added link right_wrist_yaw_link, mass 0.2; collision sphere radius=0.03; visual mesh filename=meshes/right_wrist_yaw_link.STL
- link left_ankle_roll_link: geometry collision mesh filename=meshes/left_ankle_roll_link.STL; visual mesh filename=meshes/left_ankle_roll_link.STL
- link left_elbow_link: geometry collision box size=0.10 0.04 0.04; visual mesh filename=meshes/left_elbow_link.STL
- link left_hip_yaw_link: geometry visual mesh filename=meshes/left_hip_yaw_link.STL
- link left_knee_link: geometry visual mesh filename=meshes/left_knee_link.STL
- link left_shoulder_pitch_link: geometry collision cylinder length=0.02 radius=0.02; visual mesh filename=meshes/left_shoulder_pitch_link.STL
- link left_shoulder_roll_link: geometry collision box size=0.04 0.04 0.04; visual mesh filename=meshes/left_shoulder_roll_link.STL
- link left_shoulder_yaw_link: geometry collision cylinder length=0.08 radius=0.030; visual mesh filename=meshes/left_shoulder_yaw_link.STL
- link left_wrist_pitch_link: geometry collision sphere radius=0.03; visual mesh filename=meshes/left_wrist_pitch_link.STL
- link left_wrist_roll_link: geometry collision sphere radius=0.03; visual mesh filename=meshes/left_wrist_roll_link.STL
- link pelvis: geometry collision mesh filename=meshes/pelvis.STL; visual mesh filename=meshes/pelvis.STL
- link right_ankle_roll_link: geometry collision mesh filename=meshes/right_ankle_roll_link.STL; visual mesh filename=meshes/right_ankle_roll_link.STL
- link right_elbow_link: geometry collision box size=0.10 0.04 0.04; visual mesh filename=meshes/right_elbow_link.STL
- link right_hip_yaw_link: geometry visual mesh filename=meshes/right_hip_yaw_link.STL
- link right_knee_link: geometry visual mesh filename=meshes/right_knee_link.STL
- link right_shoulder_pitch_link: geometry collision cylinder length=0.02 radius=0.02; visual mesh filename=meshes/right_shoulder_pitch_link.STL
- link right_shoulder_roll_link: geometry collision box size=0.04 0.04 0.04; visual mesh filename=meshes/right_shoulder_roll_link.STL
- link right_shoulder_yaw_link: geometry collision cylinder length=0.08 radius=0.030; visual mesh filename=meshes/right_shoulder_yaw_link.STL
- link right_wrist_pitch_link: geometry collision sphere radius=0.03; visual mesh filename=meshes/right_wrist_pitch_link.STL
- link right_wrist_roll_link: geometry collision sphere radius=0.03; visual mesh filename=meshes/right_wrist_roll_link.STL
- link torso_link: mass 8.5 -> 3.5; geometry collision mesh filename=meshes/torso_link.STL; visual mesh filename=meshes/torso_link.STL
Joints:
- added joint head_pitch_joint: type fixed, parent torso_link, child head_pitch_link, origin xyz=0 0 0.304 rpy=0 0 0, axis 0 1 0, limit lower=-0.7854 upper=1.5708 effort=14 velocity=27.28
- added joint head_yaw_joint: type fixed, parent head_pitch_link, child head_yaw_link, origin xyz=-0.01 0 0.095 rpy=0 0 0, axis 0 0 1, limit lower=-3.1415 upper=3.1415 effort=14 velocity=27.28
- added joint left_wrist_yaw_joint: type fixed, parent left_wrist_pitch_link, child left_wrist_yaw_link, origin xyz=0.07 0 0 rpy=0 0 0, axis 0 0 1, limit lower=-1.5708 upper=1.5708 effort=14 velocity=27.28
- added joint right_wrist_yaw_joint: type fixed, parent right_wrist_pitch_link, child right_wrist_yaw_link, origin xyz=0.07 0 0 rpy=0 0 0, axis 0 0 1, limit lower=-1.5708 upper=1.5708 effort=14 velocity=27.28
- joint left_ankle_pitch_joint: limit lower=-1.5708 upper=1.5708 effort=36 velocity=10.47 -> lower=-1.5708 upper=1.5708 effort=60 velocity=30.16
- joint left_ankle_roll_joint: limit lower=-1.5708 upper=1.5708 effort=14 velocity=27.28 -> lower=-1.5708 upper=1.5708 effort=14 velocity=32.99
- joint left_hip_pitch_joint: limit lower=-2.7053 upper=2.7053 effort=60 velocity=18.85 -> lower=-2.7053 upper=2.7053 effort=60 velocity=20.42
- joint left_hip_roll_joint: limit lower=-0.1745 upper=2.618 effort=36 velocity=10.47 -> lower=-0.1745 upper=2.618 effort=36 velocity=50.265
- joint left_hip_yaw_joint: limit lower=-2.4871 upper=3.0107 effort=36 velocity=10.47 -> lower=-2.4871 upper=3.0107 effort=36 velocity=50.265
- joint left_knee_joint: limit lower=0 upper=2.4435 effort=36 velocity=10.47 -> lower=0 upper=2.4435 effort=60 velocity=30.16
- joint right_ankle_pitch_joint: limit lower=-1.5708 upper=1.5708 effort=36 velocity=10.47 -> lower=-1.5708 upper=1.5708 effort=60 velocity=30.16
- joint right_ankle_roll_joint: limit lower=-1.5708 upper=1.5708 effort=14 velocity=27.28 -> lower=-1.5708 upper=1.5708 effort=14 velocity=32.99
- joint right_hip_pitch_joint: limit lower=-2.7053 upper=2.7053 effort=60 velocity=18.85 -> lower=-2.7053 upper=2.7053 effort=60 velocity=20.42
- joint right_hip_roll_joint: limit lower=-2.618 upper=0.1745 effort=36 velocity=10.47 -> lower=-2.618 upper=0.1745 effort=36 velocity=50.265
- joint right_hip_yaw_joint: limit lower=-3.0107 upper=2.4871 effort=36 velocity=10.47 -> lower=-3.0107 upper=2.4871 effort=36 velocity=50.265
- joint right_knee_joint: limit lower=0 upper=2.4435 effort=36 velocity=10.47 -> lower=0 upper=2.4435 effort=60 velocity=30.16
- joint waist_yaw_joint: limit lower=-2.618 upper=2.618 effort=14 velocity=27.28 -> lower=-2.618 upper=2.618 effort=60 velocity=20.42
