Commit message: 增加DOG模型

File: legged_lab/assets/droid/E1/E1-12.urdf (robot description, URDF)
Before this commit: robot E1_1105, 30 links, 29 joints
Links:
- link head_pitch_link: geometry visual mesh filename=meshes/head_pitch_link.STL
- link head_yaw_link: geometry collision box size=0.10 0.13 0.12; visual mesh filename=meshes/head_yaw_link.STL
- link left_ankle_roll_link: geometry collision box size=0.18 0.07 0.025; visual mesh filename=meshes/left_ankle_roll_link.STL
- link left_elbow_link: geometry collision cylinder length=0.05 radius=0.045; visual mesh filename=meshes/left_elbow_link.STL
- link left_hip_yaw_link: geometry collision cylinder length=0.2 radius=0.06; visual mesh filename=meshes/left_hip_yaw_link.STL
- link left_knee_link: geometry collision cylinder length=0.23 radius=0.045; visual mesh filename=meshes/left_knee_link.STL
- link left_shoulder_pitch_link: geometry visual mesh filename=meshes/left_shoulder_pitch_link.STL
- link left_shoulder_roll_link: geometry collision cylinder length=0.05 radius=0.044; visual mesh filename=meshes/left_shoulder_roll_link.STL
- link left_shoulder_yaw_link: geometry collision cylinder length=0.09 radius=0.045; visual mesh filename=meshes/left_shoulder_yaw_link.STL
- link left_wrist_pitch_link: geometry collision sphere radius=0.038; visual mesh filename=meshes/left_wrist_pitch_link.STL
- link left_wrist_roll_link: geometry visual mesh filename=meshes/left_wrist_roll_link.STL
- link left_wrist_yaw_link: geometry visual mesh filename=meshes/left_wrist_yaw_link.STL
- link pelvis: geometry visual mesh filename=meshes/pelvis.STL
- link right_ankle_roll_link: geometry collision box size=0.18 0.07 0.025; visual mesh filename=meshes/right_ankle_roll_link.STL
- link right_elbow_link: geometry collision cylinder length=0.05 radius=0.045; visual mesh filename=meshes/right_elbow_link.STL
- link right_hip_yaw_link: geometry collision cylinder length=0.2 radius=0.06; visual mesh filename=meshes/right_hip_yaw_link.STL
- link right_knee_link: geometry collision cylinder length=0.23 radius=0.045; visual mesh filename=meshes/right_knee_link.STL
- link right_shoulder_pitch_link: geometry visual mesh filename=meshes/right_shoulder_pitch_link.STL
- link right_shoulder_roll_link: geometry collision cylinder length=0.05 radius=0.044; visual mesh filename=meshes/right_shoulder_roll_link.STL
- link right_shoulder_yaw_link: geometry collision cylinder length=0.09 radius=0.045; visual mesh filename=meshes/right_shoulder_yaw_link.STL
- link right_wrist_pitch_link: geometry collision sphere radius=0.038; visual mesh filename=meshes/right_wrist_pitch_link.STL
- link right_wrist_roll_link: geometry visual mesh filename=meshes/right_wrist_roll_link.STL
- link right_wrist_yaw_link: geometry visual mesh filename=meshes/right_wrist_yaw_link.STL
- link torso_link: mass 3.5 -> 6.5; geometry collision box size=0.16 0.16 0.30; visual mesh filename=meshes/torso_link.STL
Joints:
- joint left_ankle_pitch_joint: limit lower=-1.5708 upper=1.5708 effort=60 velocity=30.16 -> lower=-0.87 upper=0.35 effort=36 velocity=50.265
- joint left_ankle_roll_joint: limit lower=-1.5708 upper=1.5708 effort=42 velocity=10.99 -> lower=-0.44 upper=0.44 effort=14 velocity=32.99
- joint left_hip_pitch_joint: limit lower=-2.7053 upper=2.7053 effort=60 velocity=20.42 -> lower=-1.8 upper=1.57 effort=36 velocity=50.265
- joint left_hip_roll_joint: limit lower=-0.1745 upper=2.618 effort=36 velocity=50.265 -> lower=-0.1745 upper=1.57 effort=60 velocity=20.42
- joint left_hip_yaw_joint: limit lower=-2.4871 upper=3.0107 effort=36 velocity=50.265 -> lower=-1.0 upper=1.0 effort=36 velocity=50.265
- joint right_ankle_pitch_joint: limit lower=-1.5708 upper=1.5708 effort=60 velocity=30.16 -> lower=-0.87 upper=0.35 effort=36 velocity=50.265
- joint right_ankle_roll_joint: limit lower=-1.5708 upper=1.5708 effort=42 velocity=10.99 -> lower=-0.44 upper=0.44 effort=14 velocity=32.99
- joint right_hip_pitch_joint: limit lower=-2.7053 upper=2.7053 effort=60 velocity=20.42 -> lower=-1.8 upper=1.57 effort=36 velocity=50.265
- joint right_hip_roll_joint: limit lower=-2.618 upper=0.1745 effort=36 velocity=50.265 -> lower=-1.57 upper=0.1745 effort=60 velocity=20.42
- joint right_hip_yaw_joint: limit lower=-3.0107 upper=2.4871 effort=36 velocity=50.265 -> lower=-1.0 upper=1.0 effort=36 velocity=50.265
- joint waist_yaw_joint: limit lower=-2.618 upper=2.618 effort=60 velocity=20.42 -> lower=-1.57 upper=1.57 effort=60 velocity=20.42; type revolute -> fixed
