Commit message: E1新模型测试ok

File: legged_lab/assets/droid/E1/E1.urdf (robot description, URDF)
Before this commit: robot E1, 20 links, 19 joints
Joints:
- joint left_ankle_pitch_joint: limit lower=-1.571 upper=1.571 effort=60 velocity=260 -> lower=-1.571 upper=1.571 effort=60 velocity=50
- joint left_ankle_roll_joint: limit lower=-0.524 upper=0.524 effort=60 velocity=260 -> lower=-0.524 upper=0.524 effort=60 velocity=50
- joint left_hip_pitch_joint: limit lower=-2.09 upper=0.916 effort=60 velocity=180 -> lower=-2.09 upper=0.916 effort=60 velocity=50
- joint left_hip_roll_joint: limit lower=-0.5236 upper=1.57 effort=60 velocity=180 -> lower=-0.5236 upper=1.57 effort=60 velocity=50
- joint left_hip_yaw_joint: limit lower=-2.0944 upper=2.0944 effort=60 velocity=260 -> lower=-2.0944 upper=2.0944 effort=14 velocity=50
- joint left_knee_joint: limit lower=0 upper=2.09 effort=60 velocity=260 -> lower=0 upper=2.09 effort=60 velocity=50
- joint right_ankle_pitch_joint: limit lower=-1.571 upper=1.571 effort=60 velocity=260 -> lower=-1.571 upper=1.571 effort=60 velocity=50
- joint right_ankle_roll_joint: limit lower=-0.524 upper=0.524 effort=60 velocity=260 -> lower=-0.524 upper=0.524 effort=60 velocity=50
- joint right_hip_pitch_joint: limit lower=-2.09 upper=0.916 effort=60 velocity=180 -> lower=-2.09 upper=0.916 effort=60 velocity=50
- joint right_hip_roll_joint: limit lower=-1.57 upper=0.5236 effort=60 velocity=180 -> lower=-1.57 upper=0.5236 effort=60 velocity=50
- joint right_hip_yaw_joint: limit lower=-2.0944 upper=2.0944 effort=60 velocity=260 -> lower=-2.0944 upper=2.0944 effort=14 velocity=50
- joint right_knee_joint: limit lower=0 upper=2.09 effort=60 velocity=260 -> lower=0 upper=2.09 effort=60 velocity=50

Commit message: E1新模型测试ok

File: legged_lab/assets/droid/E1/E1.urdf (robot description, URDF)
Before this commit: robot E1, 20 links, 19 joints
Links:
- added link head_pitch_link, mass 0.4; collision mesh filename=meshes/head_pitch_link.STL; visual mesh filename=meshes/head_pitch_link.STL
- added link head_yaw_link, mass 1; collision mesh filename=meshes/head_yaw_link.STL; visual mesh filename=meshes/head_yaw_link.STL
- added link left_elbow_link, mass 0.35; collision mesh filename=meshes/left_elbow_link.STL; visual mesh filename=meshes/left_elbow_link.STL
- added link left_wrist_pitch_link; collision mesh filename=meshes/left_wrist_pitch_link.STL; visual mesh filename=meshes/left_wrist_pitch_link.STL
- added link left_wrist_roll_link, mass 0.1; collision mesh filename=meshes/left_wrist_roll_link.STL; visual mesh filename=meshes/left_wrist_roll_link.STL
- added link left_wrist_yaw_link, mass 0.2; collision mesh filename=meshes/left_wrist_yaw_link.STL; visual mesh filename=meshes/left_wrist_yaw_link.STL
- added link right_elbow_link, mass 0.35; collision mesh filename=meshes/right_elbow_link.STL; visual mesh filename=meshes/right_elbow_link.STL
- added link right_wrist_pitch_link; collision mesh filename=meshes/right_wrist_pitch_link.STL; visual mesh filename=meshes/right_wrist_pitch_link.STL
- added link right_wrist_roll_link, mass 0.1; collision mesh filename=meshes/right_wrist_roll_link.STL; visual mesh filename=meshes/right_wrist_roll_link.STL
- added link right_wrist_yaw_link, mass 0.2; collision mesh filename=meshes/right_wrist_yaw_link.STL; visual mesh filename=meshes/right_wrist_yaw_link.STL
- added link waist_yaw_link, mass 0.90; collision mesh filename=meshes/waist_yaw_link.STL; visual mesh filename=meshes/waist_yaw_link.STL
- link left_ankle_pitch_link: mass 0.8 -> 0.597; geometry collision mesh filename=meshes/left_ankle_pitch_link.STL; visual mesh filename=meshes/left_ankle_pitch_link.STL
- link left_ankle_roll_link: mass 0.5 -> 0.294; geometry collision mesh filename=meshes/left_ankle_roll_link.STL; visual mesh filename=meshes/left_ankle_roll_link.STL
- link left_hip_pitch_link: mass 1.276 -> 0.145; geometry visual mesh filename=meshes/left_hip_pitch_link.STL
- link left_hip_roll_link: mass 1.126 -> 1.39; geometry visual mesh filename=meshes/left_hip_roll_link.STL
- link left_hip_yaw_link: mass 0.896 -> 2.39; geometry collision mesh filename=meshes/left_hip_yaw_link.STL; visual mesh filename=meshes/left_hip_yaw_link.STL
- link left_knee_link: mass 0.8 -> 0.785; geometry visual mesh filename=meshes/left_knee_link.STL
- link left_shoulder_pitch_link: mass 1.276 -> 0.8; geometry collision mesh filename=meshes/left_shoulder_pitch_link.STL; visual mesh filename=meshes/left_shoulder_pitch_link.STL
- link left_shoulder_roll_link: mass 1.126 -> 0.2; geometry collision mesh filename=meshes/left_shoulder_roll_link.STL; visual mesh filename=meshes/left_shoulder_roll_link.STL
- link left_shoulder_yaw_link: mass 0.896 -> 0.6; geometry collision mesh filename=meshes/left_shoulder_yaw_link.STL; visual mesh filename=meshes/left_shoulder_yaw_link.STL
- link pelvis: mass 3 -> 2.73; geometry collision mesh filename=meshes/pelvis.STL; visual mesh filename=meshes/pelvis.STL
- link right_ankle_pitch_link: mass 0.8 -> 0.597; geometry collision mesh filename=meshes/right_ankle_pitch_link.STL; visual mesh filename=meshes/right_ankle_pitch_link.STL
- link right_ankle_roll_link: mass 0.5 -> 0.294; geometry collision mesh filename=meshes/right_ankle_roll_link.STL; visual mesh filename=meshes/right_ankle_roll_link.STL
- link right_hip_pitch_link: mass 1.276 -> 0.145; geometry visual mesh filename=meshes/right_hip_pitch_link.STL
- link right_hip_roll_link: mass 1.126 -> 1.39; geometry visual mesh filename=meshes/right_hip_roll_link.STL
- link right_hip_yaw_link: mass 0.896 -> 2.39; geometry collision mesh filename=meshes/right_hip_yaw_link.STL; visual mesh filename=meshes/right_hip_yaw_link.STL
- link right_knee_link: mass 0.8 -> 0.785; geometry visual mesh filename=meshes/right_knee_link.STL
- link right_shoulder_pitch_link: mass 1.276 -> 0.8; geometry collision mesh filename=meshes/right_shoulder_pitch_link.STL; visual mesh filename=meshes/right_shoulder_pitch_link.STL
- link right_shoulder_roll_link: mass 1.126 -> 0.2; geometry collision mesh filename=meshes/right_shoulder_roll_link.STL; visual mesh filename=meshes/right_shoulder_roll_link.STL
- link right_shoulder_yaw_link: mass 0.896 -> 0.6; geometry collision mesh filename=meshes/right_shoulder_yaw_link.STL; visual mesh filename=meshes/right_shoulder_yaw_link.STL
- link torso_link: mass 6 -> 5.0; geometry collision mesh filename=meshes/torso_link.STL; visual mesh filename=meshes/torso_link.STL
Joints:
- removed joint left_shoulder_yaw_joint
- added joint head_pitch_joint: type fixed, parent torso_link, child head_pitch_link, origin xyz=0 0 0.304 rpy=0 0 0, axis 0 1 0, limit lower=-0.7854 upper=1.5708 effort=14 velocity=27.28
- added joint head_yaw_joint: type fixed, parent head_pitch_link, child head_yaw_link, origin xyz=-0.01 0 0.095 rpy=0 0 0, axis 0 0 1, limit lower=-3.1415 upper=3.1415 effort=14 velocity=27.28
- added joint left_elbow_joint: type fixed, parent left_shoulder_yaw_link, child left_elbow_link, origin xyz=0 0 -0.159 rpy=0 0 0, axis 0 1 0, limit lower=-0.6981 upper=1.5708 effort=28 velocity=27.28
- added joint left_shoulder_yaw_join: type fixed, parent left_shoulder_roll_link, child left_shoulder_yaw_link, origin xyz=0 0 -0.051 rpy=0 0 0, axis 0 0 1, limit lower=-2.618 upper=2.618 effort=14 velocity=27.28
- added joint left_wrist_pitch_joint: type fixed, parent left_wrist_roll_link, child left_wrist_pitch_link, origin xyz=0.035 0 0 rpy=0 0 0, axis 0 1 0, limit lower=-0.6109 upper=0.6109 effort=14 velocity=27.28
- added joint left_wrist_roll_joint: type fixed, parent left_elbow_link, child left_wrist_roll_link, origin xyz=0.125 0 0 rpy=0 0 0, axis 1 0 0, limit lower=-2.1817 upper=2.1817 effort=36 velocity=10.47
- added joint left_wrist_yaw_joint: type fixed, parent left_wrist_pitch_link, child left_wrist_yaw_link, origin xyz=0.07 0 0 rpy=0 0 0, axis 0 0 1, limit lower=-1.5708 upper=1.5708 effort=14 velocity=27.28
- added joint right_elbow_joint: type fixed, parent right_shoulder_yaw_link, child right_elbow_link, origin xyz=0 0 -0.159 rpy=0 0 0, axis 0 1 0, limit lower=-0.6981 upper=1.5708 effort=36 velocity=10.47
- added joint right_wrist_pitch_joint: type fixed, parent right_wrist_roll_link, child right_wrist_pitch_link, origin xyz=0.035 0 0 rpy=0 0 0, axis 0 1 0, limit lower=-0.6109 upper=0.6109 effort=14 velocity=27.28
- added joint right_wrist_roll_joint: type fixed, parent right_elbow_link, child right_wrist_roll_link, origin xyz=0.125 0 0 rpy=0 0 0, axis 1 0 0, limit lower=-2.1817 upper=2.1817 effort=14 velocity=27.28
- added joint right_wrist_yaw_joint: type fixed, parent right_wrist_pitch_link, child right_wrist_yaw_link, origin xyz=0.07 0 0 rpy=0 0 0, axis 0 0 1, limit lower=-1.5708 upper=1.5708 effort=14 velocity=27.28
- added joint waist_yaw_joint: type revolute, parent pelvis, child waist_yaw_link, origin xyz=0 0 0.111 rpy=0 0 0, axis 0 0 1, limit lower=-1.5708 upper=1.5708 effort=60 velocity=50.265
- joint left_ankle_pitch_joint: limit lower=-1.571 upper=1.571 effort=60 velocity=50 -> lower=-0.5236 upper=0.5236 effort=36 velocity=50.265; origin xyz=0 0 -0.035 rpy=0 0 0 -> xyz=0 0 -0.32 rpy=0 0 0; parent left_ankle_roll_link -> left_knee_link
- joint left_ankle_roll_joint: limit lower=-0.524 upper=0.524 effort=60 velocity=50 -> lower=-1.5708 upper=1.5708 effort=14 velocity=32.987; origin xyz=0.01 0 -0.21 rpy=0 0 0 -> xyz=0 0 -0.06 rpy=0 0 0; parent left_knee_link -> left_ankle_pitch_link
- joint left_hip_pitch_joint: limit lower=-2.09 upper=0.916 effort=60 velocity=50 -> lower=-2.7053 upper=2.7053 effort=60 velocity=20.42; origin xyz=0 0.064 0 rpy=0 0 0 -> xyz=0 0.0575 0 rpy=0 0 0
- joint left_hip_roll_joint: limit lower=-0.5236 upper=1.57 effort=60 velocity=50 -> lower=-0.5236 upper=3.1416 effort=36 velocity=50.265; origin xyz=0 0.0585 0 rpy=0 0 0 -> xyz=0 0.0575 -0.015 rpy=0 0 0
- joint left_hip_yaw_joint: limit lower=-2.0944 upper=2.0944 effort=14 velocity=50 -> lower=-2.0944 upper=2.0944 effort=36 velocity=50.265; origin xyz=0 0.015 -0.0845 rpy=0 0 0 -> xyz=0 0 -0.098 rpy=0 0 0
- joint left_knee_joint: limit lower=0 upper=2.09 effort=60 velocity=50 -> lower=0 upper=2.2689 effort=36 velocity=50.265; origin xyz=-0.01 0 -0.1605 rpy=0 0 0 -> xyz=0 0 -0.222 rpy=0 0 0
- joint left_shoulder_pitch_joint: limit lower=-4.058 upper=0.916 effort=60 velocity=180 -> lower=-1.0472 upper=2.7925 effort=36 velocity=10.47; origin xyz=0 0.13613 0.37182 rpy=0.17453 0 0 -> xyz=0 0.095 0.239 rpy=0 0 0
- joint left_shoulder_roll_joint: limit lower=0 upper=3.1416 effort=60 velocity=180 -> lower=-0.1745 upper=2.9671 effort=36 velocity=10.47; origin xyz=0 0.045976 0 rpy=-0.17453 0 0 -> xyz=0 0.055 0 rpy=0 0 0
- joint right_ankle_pitch_joint: limit lower=-1.571 upper=1.571 effort=60 velocity=50 -> lower=-0.5236 upper=0.5236 effort=36 velocity=50.265; origin xyz=0 0 -0.035 rpy=0 0 0 -> xyz=0 0 -0.32 rpy=0 0 0; parent right_ankle_roll_link -> right_knee_link
- joint right_ankle_roll_joint: limit lower=-0.524 upper=0.524 effort=60 velocity=50 -> lower=-1.5708 upper=1.5708 effort=14 velocity=27.28; origin xyz=0.01 0 -0.21 rpy=0 0 0 -> xyz=0 0 -0.06 rpy=0 0 0; parent right_knee_link -> right_ankle_pitch_link
- joint right_hip_pitch_joint: limit lower=-2.09 upper=0.916 effort=60 velocity=50 -> lower=-2.7053 upper=2.7053 effort=60 velocity=20.42; origin xyz=0 -0.064 0 rpy=0 0 0 -> xyz=0 -0.0575 0 rpy=0 0 0
- joint right_hip_roll_joint: limit lower=-1.57 upper=0.5236 effort=60 velocity=50 -> lower=-2.618 upper=0.1745 effort=36 velocity=50.265; origin xyz=0 -0.0585 0 rpy=0 0 0 -> xyz=0 -0.0575 -0.015 rpy=0 0 0
- joint right_hip_yaw_joint: limit lower=-2.0944 upper=2.0944 effort=14 velocity=50 -> lower=-2.0944 upper=2.0944 effort=36 velocity=50.265; origin xyz=0 -0.015 -0.0845 rpy=0 0 0 -> xyz=0 0 -0.098 rpy=0 0 0
- joint right_knee_joint: limit lower=0 upper=2.09 effort=60 velocity=50 -> lower=0 upper=2.2689 effort=36 velocity=50.265; origin xyz=-0.01 0 -0.1605 rpy=0 0 0 -> xyz=0 0 -0.222 rpy=0 0 0
- joint right_shoulder_pitch_joint: limit lower=-4.058 upper=0.916 effort=60 velocity=180 -> lower=-1.0472 upper=2.7925 effort=36 velocity=10.47; origin xyz=0 -0.13615 0.37182 rpy=-0.17453 0 0 -> xyz=0 -0.095 0.239 rpy=0 0 0
- joint right_shoulder_roll_joint: limit lower=-3.1416 upper=0 effort=60 velocity=180 -> lower=-2.9671 upper=0.1745 effort=36 velocity=10.47; origin xyz=0 -0.045957 0 rpy=0.17453 0 0 -> xyz=0 -0.055 0 rpy=0 0 0
- joint right_shoulder_yaw_joint: limit lower=-2.0944 upper=2.0944 effort=5 velocity=260 -> lower=-2.618 upper=2.618 effort=14 velocity=27.28; origin xyz=0 -0.015 -0.0845 rpy=0 0 0 -> xyz=0 0 -0.051 rpy=0 0 0
- joint torso_joint: parent pelvis -> waist_yaw_link

File: legged_lab/assets/droid/X2C_PRO/X2C_PRO_pink.urdf (robot description, URDF)
Before this commit: robot X02C_PRO, 26 links, 25 joints
Links:
- added link world
Joints:
- added joint pelvis_link: type floating, parent world, child pelvis_link

Commit message: E1新模型测试ok

File: legged_lab/assets/droid/E1/E1.urdf (robot description, URDF)
Before this commit: robot E1_1105, 31 links, 30 joints
Links:
- removed link head_pitch_link
- removed link head_yaw_link
- removed link left_wrist_yaw_link
- removed link right_wrist_yaw_link
- removed link waist_yaw_link
- link left_ankle_pitch_link: geometry visual mesh filename=meshes/left_ankle_pitch_link.STL
- link left_ankle_roll_link: geometry collision box size=0.18 0.06 0.04; visual mesh filename=meshes/left_ankle_roll_link.STL
- link left_elbow_link: mass 0.35 -> 0.51; geometry visual mesh filename=meshes/left_elbow_link.STL
- link left_hip_yaw_link: mass 2.39 -> 2.32; geometry collision cylinder length=0.10 radius=0.04; visual mesh filename=meshes/left_hip_yaw_link.STL
- link left_knee_link: geometry collision box size=0.06 0.06 0.2; visual mesh filename=meshes/left_knee_link.STL
- link left_shoulder_pitch_link: mass 0.8 -> 0.86; geometry visual mesh filename=meshes/left_shoulder_pitch_link.STL
- link left_shoulder_roll_link: mass 0.2 -> 0.1; geometry visual mesh filename=meshes/left_shoulder_roll_link.STL
- link left_shoulder_yaw_link: mass 0.6 -> 1.55; geometry visual mesh filename=meshes/left_shoulder_yaw_link.STL
- link left_wrist_pitch_link: mass None -> 0.005; geometry visual mesh filename=meshes/left_wrist_pitch_link.STL
- link left_wrist_roll_link: mass 0.1 -> 0.38; geometry visual mesh filename=meshes/left_wrist_roll_link.STL
- link pelvis: geometry visual mesh filename=meshes/pelvis.STL
- link right_ankle_pitch_link: geometry visual mesh filename=meshes/right_ankle_pitch_link.STL
- link right_ankle_roll_link: geometry collision box size=0.18 0.06 0.04; visual mesh filename=meshes/right_ankle_roll_link.STL
- link right_elbow_link: mass 0.35 -> 0.51; geometry visual mesh filename=meshes/right_elbow_link.STL
- link right_hip_yaw_link: mass 2.39 -> 2.32; geometry collision cylinder length=0.10 radius=0.04; visual mesh filename=meshes/right_hip_yaw_link.STL
- link right_knee_link: geometry collision box size=0.06 0.06 0.2; visual mesh filename=meshes/right_knee_link.STL
- link right_shoulder_pitch_link: mass 0.8 -> 0.86; geometry visual mesh filename=meshes/right_shoulder_pitch_link.STL
- link right_shoulder_roll_link: mass 0.2 -> 0.1; geometry visual mesh filename=meshes/right_shoulder_roll_link.STL
- link right_shoulder_yaw_link: mass 0.6 -> 1.55; geometry visual mesh filename=meshes/right_shoulder_yaw_link.STL
- link right_wrist_pitch_link: mass None -> 0.005; geometry visual mesh filename=meshes/right_wrist_pitch_link.STL
- link right_wrist_roll_link: mass 0.1 -> 0.38; geometry visual mesh filename=meshes/right_wrist_roll_link.STL
- link torso_link: mass 5.0 -> 8.5; geometry collision box size=0.16 0.16 0.30; visual mesh filename=meshes/torso_link.STL
Joints:
- removed joint head_pitch_joint
- removed joint head_yaw_joint
- removed joint left_shoulder_yaw_join
- removed joint left_wrist_yaw_joint
- removed joint right_wrist_yaw_joint
- removed joint torso_joint
- added joint left_shoulder_yaw_joint: type fixed, parent left_shoulder_roll_link, child left_shoulder_yaw_link, origin xyz=0 0 -0.051 rpy=0 0 0, axis 0 0 1, limit lower=-2.618 upper=2.618 effort=14 velocity=27.28
- joint left_ankle_pitch_joint: limit lower=-0.5236 upper=0.5236 effort=36 velocity=50.265 -> lower=-1.5708 upper=1.5708 effort=36 velocity=10.47
- joint left_ankle_roll_joint: limit lower=-1.5708 upper=1.5708 effort=14 velocity=32.987 -> lower=-1.5708 upper=1.5708 effort=14 velocity=27.28
- joint left_hip_pitch_joint: limit lower=-2.7053 upper=2.7053 effort=60 velocity=20.42 -> lower=-2.7053 upper=2.7053 effort=60 velocity=18.85
- joint left_hip_roll_joint: limit lower=-0.5236 upper=3.1416 effort=36 velocity=50.265 -> lower=-0.1745 upper=2.618 effort=36 velocity=10.47
- joint left_hip_yaw_joint: limit lower=-2.0944 upper=2.0944 effort=36 velocity=50.265 -> lower=-2.4871 upper=3.0107 effort=36 velocity=10.47
- joint left_knee_joint: limit lower=0 upper=2.2689 effort=36 velocity=50.265 -> lower=0 upper=2.4435 effort=36 velocity=10.47
- joint right_ankle_pitch_joint: limit lower=-0.5236 upper=0.5236 effort=36 velocity=50.265 -> lower=-1.5708 upper=1.5708 effort=36 velocity=10.47
- joint right_hip_pitch_joint: limit lower=-2.7053 upper=2.7053 effort=60 velocity=20.42 -> lower=-2.7053 upper=2.7053 effort=60 velocity=18.85
- joint right_hip_roll_joint: limit lower=-2.618 upper=0.1745 effort=36 velocity=50.265 -> lower=-2.618 upper=0.1745 effort=36 velocity=10.47
- joint right_hip_yaw_joint: limit lower=-2.0944 upper=2.0944 effort=36 velocity=50.265 -> lower=-3.0107 upper=2.4871 effort=36 velocity=10.47
- joint right_knee_joint: limit lower=0 upper=2.2689 effort=36 velocity=50.265 -> lower=0 upper=2.4435 effort=36 velocity=10.47
- joint waist_yaw_joint: child waist_yaw_link -> torso_link; limit lower=-1.5708 upper=1.5708 effort=60 velocity=50.265 -> lower=-2.618 upper=2.618 effort=14 velocity=27.28

Commit message: E1_DOG Sim2Real验证完成

File: legged_lab/assets/droid/E1/E1.urdf (robot description, URDF)
Before this commit: robot E1_1105, 30 links, 29 joints
Joints:
- joint waist_yaw_joint: type revolute -> fixed

File: legged_lab/assets/droid/E1_DOG/E1_DOG.urdf (robot description, URDF)
Before this commit: robot E1dog, 20 links, 19 joints
Links:
- link base: mass 6 -> 4

Commit message: 完善了从训练到部署的全流程

File: legged_lab/assets/droid/E1/E1.urdf (robot description, URDF)
Before this commit: robot E1_1105, 30 links, 29 joints
Links:
- removed link head_pitch_link
- removed link head_yaw_link
- removed link left_elbow_link
- removed link left_wrist_pitch_link
- removed link left_wrist_roll_link
- removed link left_wrist_yaw_link
- removed link right_elbow_link
- removed link right_wrist_pitch_link
- removed link right_wrist_roll_link
- removed link right_wrist_yaw_link
- link left_ankle_roll_link: geometry collision sphere radius=0.005; collision sphere radius=0.005
- link left_hip_yaw_link: mass 2.32 -> 2.39
- link left_knee_link: mass 0.785 -> 1.408; geometry collision mesh filename=meshes/left_knee_link.STL; visual mesh filename=meshes/left_knee_link.STL
- link left_shoulder_pitch_link: mass 0.86 -> 0.7; geometry visual mesh filename=meshes/left_shoulder_pitch_link.STL
- link left_shoulder_roll_link: geometry visual mesh filename=meshes/left_shoulder_roll_link.STL
- link left_shoulder_yaw_link: mass 1.55 -> 1.366; geometry visual mesh filename=meshes/left_shoulder_yaw_link.STL
- link pelvis: mass 2.73 -> 3.5
- link right_ankle_roll_link: geometry collision sphere radius=0.005; collision sphere radius=0.005
- link right_hip_yaw_link: mass 2.32 -> 2.39
- link right_knee_link: mass 0.785 -> 1.408; geometry collision mesh filename=meshes/right_knee_link.STL; visual mesh filename=meshes/right_knee_link.STL
- link right_shoulder_pitch_link: mass 0.86 -> 0.7; geometry visual mesh filename=meshes/right_shoulder_pitch_link.STL
- link right_shoulder_roll_link: geometry visual mesh filename=meshes/right_shoulder_roll_link.STL
- link right_shoulder_yaw_link: mass 1.55 -> 1.366; geometry visual mesh filename=meshes/right_shoulder_yaw_link.STL
- link torso_link: mass 3.5 -> 6; geometry collision box size=0.16 0.16 0.30; visual mesh filename=meshes/torso_link.STL
Joints:
- removed joint head_pitch_joint
- removed joint head_yaw_joint
- removed joint left_elbow_joint
- removed joint left_wrist_pitch_joint
- removed joint left_wrist_roll_joint
- removed joint left_wrist_yaw_joint
- removed joint right_elbow_joint
- removed joint right_wrist_pitch_joint
- removed joint right_wrist_roll_joint
- removed joint right_wrist_yaw_joint
- joint left_ankle_roll_joint: limit lower=-1.5708 upper=1.5708 effort=42 velocity=10.99 -> lower=-1.5708 upper=1.5708 effort=14 velocity=32.99
- joint right_ankle_roll_joint: limit lower=-1.5708 upper=1.5708 effort=42 velocity=10.99 -> lower=-1.5708 upper=1.5708 effort=14 velocity=32.99

File: legged_lab/assets/droid/E1_DOG/E1_DOG.urdf (robot description, URDF)
Before this commit: robot E1dog, 20 links, 19 joints
Joints:
- joint FL_foot_joint: axis (none) -> 0 0 0
- joint FR_foot_joint: axis (none) -> 0 0 0
- joint RL_foot_joint: axis (none) -> 0 0 0
- joint RR_foot_joint: axis (none) -> 0 0 0
